Commit message: Finally make manipulator proper work

File: simulation_ws/src/mrm_description/urdf/mrm.xacro (robot description, xacro)
@@ -1,26 +1,48 @@
 <?xml version="1.0" ?>
 <robot name="mrm" xmlns:xacro="http://www.ros.org/wiki/xacro">
-    <link name="base_link">
-        <visual>
-            <origin rpy="0 0 0" xyz="0 0 0"/>
-            <geometry>
-                <box size="1 1 1"/>
-            </geometry>
-        </visual>
-    </link>
-    <joint name="base_link__link_01" type="revolute">
-        <axis xyz="0 0 1" />
-        <limit effort="1000.0" lower="-3.14" upper="3.14" velocity="0.5" />
-        <origin rpy="0 0 0" xyz="0 0 0.5"/>
-        <parent link="base_link"/>
-        <child link="link1"/>
-    </joint>
-    <link name="link1">
-        <visual>
-            <origin rpy="0 0 0" xyz="0 0 0.2"/>
-            <geometry>
-                <cylinder radius="0.35" length="0.4"/>
-            </geometry>
-        </visual>
-    </link>
+  <!-- BGN - Include -->
+  <xacro:include filename="$(find mrm_description)/urdf/links_joints.xacro" />
+  <xacro:include filename="$(find mrm_description)/urdf/robot_parameters.xacro" />
+  <!-- END - Include -->
+  <!-- BGN - Robot description -->
+  <xacro:m_link_box name="${link_00_name}"
+              origin_rpy="0 0 0" origin_xyz="0 0 0"
+              size="1 1 1" />
+  <xacro:m_joint name="${link_00_name}__${link_01_name}" type="revolute"
+           axis_xyz="0 0 1"
+           origin_rpy="0 0 0" origin_xyz="0 0 0.5"
+           parent="${link_00_name}" child="${link_01_name}" />
+  <xacro:m_link_cylinder name="${link_01_name}"
+              origin_rpy="0 0 0" origin_xyz="0 0 0.2"
+              length="0.4" radius="0.35" />
+  <xacro:m_joint name="${link_01_name}__${link_02_name}" type="revolute"
+           axis_xyz="0 1 0"
+           origin_rpy="0 0 0" origin_xyz="0 0 0.4"
+           parent="${link_01_name}" child="${link_02_name}" />
+  <xacro:m_link_cylinder name="${link_02_name}"
+              origin_rpy="0 0 0" origin_xyz="0 0 0.4"
+              radius="0.15" length="0.8" />
+  <xacro:m_joint name="${link_02_name}__${link_03_name}" type="revolute"
+           axis_xyz="0 1 0"
+           origin_rpy="0 0 0" origin_xyz="0 0 0.8"
+           parent="${link_02_name}" child="${link_03_name}" />
+  <xacro:m_link_cylinder name="${link_03_name}"
+              origin_rpy="0 0 0" origin_xyz="0 0 0.4"
+              radius="0.15" length="0.8" />
+  <xacro:m_joint name="${link_03_name}__${link_04_name}" type="revolute"
+           axis_xyz="0 1 0"
+           origin_rpy="0 0 0" origin_xyz="0 0 0.8"
+           parent="${link_03_name}" child="${link_04_name}" />
+  <xacro:m_link_cylinder name="${link_04_name}"
+              origin_rpy="0 0 0" origin_xyz="0 0 0.4"
+              radius="0.15" length="0.8" />
+  <xacro:m_joint name="${link_04_name}__${link_05_name}" type="revolute"
+           axis_xyz="0 0 1"
+           origin_rpy="0 0 0" origin_xyz="0 0 0.8"
+           parent="${link_04_name}" child="${link_05_name}" />
+  <xacro:m_link_cylinder name="${link_05_name}"
+              origin_rpy="0 0 0" origin_xyz="0 0 0.125"
+              radius="0.15" length="0.25" />
+  <!-- END - Robot description -->
 </robot>
+<!-- https://www.theconstructsim.com/my-robotic-manipulator-02-urdf-xacro/ -->

Commit message: Make effort-controller and add transition to the model.

File: simulation_ws/src/mrm_description/urdf/mrm.xacro (robot description, xacro)
@@ -17,4 +17,14 @@
            origin_rpy="0 0 0" origin_xyz="0 0 0.5"
            parent="${link_00_name}" child="${link_01_name}" />
+  <transmission name="trans_${link_00_name}__${link_01_name}">
+    <type>transmission_interface/SimpleTransmission</type>
+    <joint name="${link_00_name}__${link_01_name}">
+        <hardwareInterface>hardware_interface/EffortJointInterface</hardwareInterface>
+    </joint>
+    <actuator name="motor_${link_00_name}__${link_01_name}">
+        <hardwareInterface>hardware_interface/EffortJointInterface</hardwareInterface>
+        <mechanicalReduction>1</mechanicalReduction>
+    </actuator>
+  </transmission>
   <xacro:m_link_cylinder name="${link_01_name}"
               origin_rpy="0 0 0" origin_xyz="0 0 0.2"
@@ -28,4 +38,14 @@
            origin_rpy="0 0 0" origin_xyz="0 0 0.4"
            parent="${link_01_name}" child="${link_02_name}" />
+  <transmission name="trans_${link_01_name}__${link_02_name}">
+    <type>transmission_interface/SimpleTransmission</type>
+    <joint name="${link_01_name}__${link_02_name}">
+        <hardwareInterface>hardware_interface/EffortJointInterface</hardwareInterface>
+    </joint>
+    <actuator name="motor_${link_01_name}__${link_02_name}">
+        <hardwareInterface>hardware_interface/EffortJointInterface</hardwareInterface>
+        <mechanicalReduction>1</mechanicalReduction>
+    </actuator>
+  </transmission>
   <xacro:m_link_cylinder name="${link_02_name}"
               origin_rpy="0 0 0" origin_xyz="0 0 0.4"
@@ -35,5 +55,5 @@
               izz="0.651"
               radius="0.15" length="0.8" />
-  <xacro:m_joint name="${link_02_name}__${link_03_name}" type="revolute"
+  <!-- <xacro:m_joint name="${link_02_name}__${link_03_name}" type="revolute"
            axis_xyz="0 1 0"
            origin_rpy="0 0 0" origin_xyz="0 0 0.8"
@@ -67,6 +87,12 @@
               iyy="0.479" iyz="0"
               izz="0.204"
-              radius="0.15" length="0.25" />
+              radius="0.15" length="0.25" /> -->
   <!-- END - Robot description -->
+<gazebo>
+  <plugin name="gazebo_ros_control" filename="libgazebo_ros_control.so">
+  </plugin>
+</gazebo>
 </robot>
 <!-- https://www.theconstructsim.com/my-robotic-manipulator-02-urdf-xacro/ -->
+<!-- How to add transmission is below -->
+<!-- https://www.theconstructsim.com/my-robotic-manipulator-04-urdf-transmission-gazebo-controllers/ -->
