Commit message: Make model inertia for gazebo simulator

File: simulation_ws/src/mrm_description/urdf/links_joints.xacro (robot description, xacro)
@@ -10,6 +10,17 @@
     </joint>
   </xacro:macro>
-  <xacro:macro name="m_link_cylinder" params="name origin_xyz origin_rpy radius length">
+  <xacro:macro name="m_link_cylinder" params="name origin_xyz origin_rpy radius length mass ixx ixy ixz iyy iyz izz">
     <link name="${name}">
+    <inertial>
+        <mass value="${mass}" />
+        <origin rpy="${origin_rpy}" xyz="${origin_xyz}" />
+        <inertia ixx="${ixx}" ixy="${ixy}" ixz="${ixz}" iyy="${iyy}" iyz="${iyz}" izz="${izz}" />
+    </inertial>
+    <collision>
+        <origin rpy="${origin_rpy}" xyz="${origin_xyz}" />
+        <geometry>
+            <cylinder radius="${radius}" length="${length}" />
+        </geometry>
+    </collision>
     <visual>
       <origin rpy="${origin_rpy}" xyz="${origin_xyz}" />
@@ -20,6 +31,17 @@
     </link>
   </xacro:macro>
-  <xacro:macro name="m_link_box" params="name origin_xyz origin_rpy size">
+  <xacro:macro name="m_link_box" params="name origin_xyz origin_rpy size mass ixx ixy ixz iyy iyz izz">
     <link name="${name}">
+    <inertial>
+        <mass value="${mass}" />
+        <origin rpy="${origin_rpy}" xyz="${origin_xyz}" />
+        <inertia ixx="${ixx}" ixy="${ixy}" ixz="${ixz}" iyy="${iyy}" iyz="${iyz}" izz="${izz}" />
+    </inertial>
+    <collision>
+        <origin rpy="${origin_rpy}" xyz="${origin_xyz}" />
+        <geometry>
+        <box size="${size}" />
+        </geometry>
+    </collision>
     <visual>
       <origin rpy="${origin_rpy}" xyz="${origin_xyz}" />

File: simulation_ws/src/mrm_description/urdf/mrm.xacro (robot description, xacro)
@@ -8,4 +8,8 @@
   <xacro:m_link_box name="${link_00_name}"
               origin_rpy="0 0 0" origin_xyz="0 0 0"
+              mass="1024"
+              ixx="170.667" ixy="0" ixz="0"
+              iyy="170.667" iyz="0"
+              izz="170.667"
               size="1 1 1" />
   <xacro:m_joint name="${link_00_name}__${link_01_name}" type="revolute"
@@ -15,4 +19,8 @@
   <xacro:m_link_cylinder name="${link_01_name}"
               origin_rpy="0 0 0" origin_xyz="0 0 0.2"
+              mass="157.633"
+              ixx="13.235" ixy="0" ixz="0"
+              iyy="13.235" iyz="0"
+              izz="9.655"
               length="0.4" radius="0.35" />
   <xacro:m_joint name="${link_01_name}__${link_02_name}" type="revolute"
@@ -22,4 +30,8 @@
   <xacro:m_link_cylinder name="${link_02_name}"
               origin_rpy="0 0 0" origin_xyz="0 0 0.4"
+              mass="57.906"
+              ixx="12.679" ixy="0" ixz="0"
+              iyy="12.679" iyz="0"
+              izz="0.651"
               radius="0.15" length="0.8" />
   <xacro:m_joint name="${link_02_name}__${link_03_name}" type="revolute"
@@ -29,4 +41,8 @@
   <xacro:m_link_cylinder name="${link_03_name}"
               origin_rpy="0 0 0" origin_xyz="0 0 0.4"
+              mass="57.906"
+              ixx="12.679" ixy="0" ixz="0"
+              iyy="12.679" iyz="0"
+              izz="0.651"
               radius="0.15" length="0.8" />
   <xacro:m_joint name="${link_03_name}__${link_04_name}" type="revolute"
@@ -36,4 +52,8 @@
   <xacro:m_link_cylinder name="${link_04_name}"
               origin_rpy="0 0 0" origin_xyz="0 0 0.4"
+              mass="57.906"
+              ixx="12.679" ixy="0" ixz="0"
+              iyy="12.679" iyz="0"
+              izz="0.651"
               radius="0.15" length="0.8" />
   <xacro:m_joint name="${link_04_name}__${link_05_name}" type="revolute"
@@ -43,4 +63,8 @@
   <xacro:m_link_cylinder name="${link_05_name}"
               origin_rpy="0 0 0" origin_xyz="0 0 0.125"
+              mass="18.056"
+              ixx="0.479" ixy="0" ixz="0"
+              iyy="0.479" iyz="0"
+              izz="0.204"
               radius="0.15" length="0.25" />
   <!-- END - Robot description -->

Commit message: Make all joints, add PID to a model.

File: simulation_ws/src/mrm_description/urdf/links_joints.xacro (robot description, xacro)
@@ -1,12 +1,22 @@
 <?xml version="1.0" ?>
 <robot xmlns:xacro="http://www.ros.org/wiki/xacro">
-  <xacro:macro name="m_joint" params="name type axis_xyz origin_rpy origin_xyz parent child">
+  <xacro:macro name="m_joint" params="name type axis_xyz origin_rpy origin_xyz parent child limit_e limit_l limit_u limit_v">
     <joint name="${name}" type="${type}">
       <axis xyz="${axis_xyz}" />
-      <limit effort="1000.0" lower="-3.14" upper="3.14" velocity="0.5" />
+      <limit effort="${limit_e}" lower="${limit_l}" upper="${limit_u}" velocity="${limit_v}" />
       <origin rpy="${origin_rpy}" xyz="${origin_xyz}" />
       <parent link="${parent}" />
       <child link="${child}" />
     </joint>
+    <transmission name="trans_${name}">
+      <type>transmission_interface/SimpleTransmission</type>
+      <joint name="${name}">
+        <hardwareInterface>hardware_interface/EffortJointInterface</hardwareInterface>
+      </joint>
+      <actuator name="motor_${name}">
+        <hardwareInterface>hardware_interface/EffortJointInterface</hardwareInterface>
+        <mechanicalReduction>1</mechanicalReduction>
+      </actuator>
+    </transmission>
   </xacro:macro>
   <xacro:macro name="m_link_cylinder" params="name origin_xyz origin_rpy radius length mass ixx ixy ixz iyy iyz izz">

File: simulation_ws/src/mrm_description/urdf/mrm.xacro (robot description, xacro)
@@ -16,15 +16,6 @@
            axis_xyz="0 0 1"
            origin_rpy="0 0 0" origin_xyz="0 0 0.5"
-           parent="${link_00_name}" child="${link_01_name}" />
-  <transmission name="trans_${link_00_name}__${link_01_name}">
-    <type>transmission_interface/SimpleTransmission</type>
-    <joint name="${link_00_name}__${link_01_name}">
-        <hardwareInterface>hardware_interface/EffortJointInterface</hardwareInterface>
-    </joint>
-    <actuator name="motor_${link_00_name}__${link_01_name}">
-        <hardwareInterface>hardware_interface/EffortJointInterface</hardwareInterface>
-        <mechanicalReduction>1</mechanicalReduction>
-    </actuator>
-  </transmission>
+           parent="${link_00_name}" child="${link_01_name}"
+           limit_e="1000" limit_l="-3.14" limit_u="3.14" limit_v="0.5" />
   <xacro:m_link_cylinder name="${link_01_name}"
               origin_rpy="0 0 0" origin_xyz="0 0 0.2"
@@ -37,15 +28,6 @@
            axis_xyz="0 1 0"
            origin_rpy="0 0 0" origin_xyz="0 0 0.4"
-           parent="${link_01_name}" child="${link_02_name}" />
-  <transmission name="trans_${link_01_name}__${link_02_name}">
-    <type>transmission_interface/SimpleTransmission</type>
-    <joint name="${link_01_name}__${link_02_name}">
-        <hardwareInterface>hardware_interface/EffortJointInterface</hardwareInterface>
-    </joint>
-    <actuator name="motor_${link_01_name}__${link_02_name}">
-        <hardwareInterface>hardware_interface/EffortJointInterface</hardwareInterface>
-        <mechanicalReduction>1</mechanicalReduction>
-    </actuator>
-  </transmission>
+           parent="${link_01_name}" child="${link_02_name}"
+           limit_e="1000" limit_l="0" limit_u="0.5" limit_v="0.5" />
   <xacro:m_link_cylinder name="${link_02_name}"
               origin_rpy="0 0 0" origin_xyz="0 0 0.4"
@@ -55,8 +37,9 @@
               izz="0.651"
               radius="0.15" length="0.8" />
-  <!-- <xacro:m_joint name="${link_02_name}__${link_03_name}" type="revolute"
+  <xacro:m_joint name="${link_02_name}__${link_03_name}" type="revolute"
            axis_xyz="0 1 0"
            origin_rpy="0 0 0" origin_xyz="0 0 0.8"
-           parent="${link_02_name}" child="${link_03_name}" />
+           parent="${link_02_name}" child="${link_03_name}"
+           limit_e="1000" limit_l="0" limit_u="0.75" limit_v="0.5" />
   <xacro:m_link_cylinder name="${link_03_name}"
               origin_rpy="0 0 0" origin_xyz="0 0 0.4"
@@ -69,5 +52,6 @@
            axis_xyz="0 1 0"
            origin_rpy="0 0 0" origin_xyz="0 0 0.8"
-           parent="${link_03_name}" child="${link_04_name}" />
+           parent="${link_03_name}" child="${link_04_name}"
+           limit_e="1000" limit_l="0" limit_u="0.75" limit_v="0.5"/>
   <xacro:m_link_cylinder name="${link_04_name}"
               origin_rpy="0 0 0" origin_xyz="0 0 0.4"
@@ -80,5 +64,6 @@
            axis_xyz="0 0 1"
            origin_rpy="0 0 0" origin_xyz="0 0 0.8"
-           parent="${link_04_name}" child="${link_05_name}" />
+           parent="${link_04_name}" child="${link_05_name}"
+           limit_e="1000" limit_l="-3.14" limit_u="3.14" limit_v="0.5" />
   <xacro:m_link_cylinder name="${link_05_name}"
               origin_rpy="0 0 0" origin_xyz="0 0 0.125"
@@ -87,5 +72,5 @@
               iyy="0.479" iyz="0"
               izz="0.204"
-              radius="0.15" length="0.25" /> -->
+              radius="0.15" length="0.25" />
   <!-- END - Robot description -->
 <gazebo>
